File: doc/pcb/LEDthermowatch/LEDthermowatch.kicad_pcb (KiCad board)
At the start: 2 copper layers, 85.6 x 54 mm, 0 parts

Commit message: drawn PCB
Parts:
- added C1: 100n, Capacitor_SMD:C_0805_2012Metric, B.Cu at (132.6, 92.4)
- added C15: 100n, Capacitor_SMD:C_0805_2012Metric, B.Cu at (182.2, 101.8)
- added C16: 100n, Capacitor_SMD:C_0805_2012Metric, B.Cu at (182.2, 110.1)
- added C17: 100n, Capacitor_SMD:C_0805_2012Metric, B.Cu at (182.3, 104.2)
- added C18: 100n, Capacitor_SMD:C_0805_2012Metric, B.Cu at (182.3, 112.2)
- added C19: 100n, Capacitor_SMD:C_0805_2012Metric, B.Cu at (116.6, 110.4)
- added C2: 100n, Capacitor_SMD:C_0805_2012Metric, B.Cu at (136.5, 88.2)
- added C20: 100n, Capacitor_SMD:C_0805_2012Metric, B.Cu at (177.2, 101.8)
- added C3: 10uF, Capacitor_THT:CP_Radial_D6.3mm_P2.50mm, F.Cu at (132.4, 81.9)
- added C4: 10uF, Capacitor_THT:CP_Radial_D6.3mm_P2.50mm, F.Cu at (118.5, 88.1)
- added C6: 100n, Capacitor_SMD:C_0805_2012Metric, B.Cu at (135.8, 83.5)
- added C7: 1u, Capacitor_THT:CP_Radial_D6.3mm_P2.50mm, F.Cu at (131.8, 68.8)
- added C8: 10p, Capacitor_SMD:C_0805_2012Metric, B.Cu at (140.0, 88.7)
- added C9: 10p, Capacitor_SMD:C_0805_2012Metric, B.Cu at (140.0, 86.6)
- added D1: LED, LED_SMD:LED_0805_2012Metric, F.Cu at (109.7, 87.6)
- added D2: LED2, LED_SMD:LED_0805_2012Metric, F.Cu at (120.6, 116.8)
- added D3: LED1, LED_SMD:LED_0805_2012Metric, F.Cu at (174.9, 98.8)
- added G***: LOGO, AE_logo:AE_logo, F.Cu at (119.0, 73.5)
- added G***: LOGO, AE_logo:RS_logo, B.Cu at (119.5, 73.5)
- added H1: MountingHole_Pad, BartLib_Pad:WirePad 4mm^2 Rect, F.Cu at (108.0, 67.0)
- added H2: MountingHole_Pad, BartLib_Pad:WirePad 4mm^2 Rect, F.Cu at (108.0, 115.2)
- added H3: MountingHole_Pad, BartLib_Pad:WirePad 4mm^2 Rect, F.Cu at (189.8, 67.0)
- added H4: MountingHole_Pad, BartLib_Pad:WirePad 4mm^2 Rect, F.Cu at (189.8, 115.2)
- added J1: Lipo L503040, BartLib_Battery:CELLEVIA 30x40mm, F.Cu at (151.0, 101.5)
- added J2: SWD, Connector_PinHeader_2.54mm:PinHeader_1x05_P2.54mm_Vertical, F.Cu at (110.9, 92.5)
- added J3: USB_B_Micro, Connector_USB:USB_Micro-B_Molex_47346-0001, B.Cu at (108.8, 80.2)
- added Q1: BC558, Package_TO_SOT_THT:TO-92, F.Cu at (173.7, 94.6)
- added Q2: BC558, Package_TO_SOT_THT:TO-92, F.Cu at (179.4, 94.6)
- added Q3: BC558, Package_TO_SOT_THT:TO-92, F.Cu at (185.0, 94.6)
- added Q4: BC558, Package_TO_SOT_THT:TO-92, F.Cu at (187.2, 88.1)
- added Q5: 2N7000, Package_TO_SOT_THT:TO-92, F.Cu at (181.0, 88.0)
- added R1: 10k, Resistor_THT:R_Axial_DIN0207_L6.3mm_D2.5mm_P10.16mm_Horizontal, B.Cu at (161.7, 108.2)
- added R10: 220, Resistor_THT:R_Axial_DIN0207_L6.3mm_D2.5mm_P10.16mm_Horizontal, B.Cu at (161.7, 114.8)
- added R11: 220, Resistor_THT:R_Axial_DIN0207_L6.3mm_D2.5mm_P10.16mm_Horizontal, B.Cu at (161.7, 111.5)
- added R14: 220R, Resistor_THT:R_Axial_DIN0207_L6.3mm_D2.5mm_P10.16mm_Horizontal, B.Cu at (171.8, 101.8)
- added R16: 1k, Resistor_THT:R_Axial_DIN0207_L6.3mm_D2.5mm_P10.16mm_Horizontal, B.Cu at (133.4, 98.5)
- added R17: 1k, Resistor_THT:R_Axial_DIN0207_L6.3mm_D2.5mm_P10.16mm_Horizontal, B.Cu at (133.4, 101.8)
- added R18: 470R, Resistor_SMD:R_0805_2012Metric, B.Cu at (152.6, 66.8)
- added R19: 470R, Resistor_SMD:R_0805_2012Metric, B.Cu at (172.0, 67.2)
- added R2: 220R, Resistor_THT:R_Axial_DIN0207_L6.3mm_D2.5mm_P10.16mm_Horizontal, B.Cu at (150.4, 71.8)
- added R20: 470R, Resistor_SMD:R_0805_2012Metric, B.Cu at (163.8, 79.2)
- added R21: 470R, Resistor_SMD:R_0805_2012Metric, B.Cu at (158.5, 79.4)
- added R22: 470R, Resistor_SMD:R_0805_2012Metric, B.Cu at (155.8, 79.2)
- added R23: 470R, Resistor_SMD:R_0805_2012Metric, B.Cu at (166.6, 72.0)
- added R24: 470R, Resistor_SMD:R_0805_2012Metric, B.Cu at (166.5, 79.2)
- added R25: 470R, Resistor_SMD:R_0805_2012Metric, B.Cu at (151.5, 86.2)
- added R26: 1k, Resistor_THT:R_Axial_DIN0207_L6.3mm_D2.5mm_P10.16mm_Horizontal, B.Cu at (159.2, 98.0)
- added R27: 1k, Resistor_THT:R_Axial_DIN0207_L6.3mm_D2.5mm_P10.16mm_Horizontal, B.Cu at (159.2, 94.8)
- added R28: 1k, Resistor_THT:R_Axial_DIN0207_L6.3mm_D2.5mm_P10.16mm_Horizontal, B.Cu at (159.2, 91.5)
- added R29: 1k, Resistor_THT:R_Axial_DIN0207_L6.3mm_D2.5mm_P10.16mm_Horizontal, B.Cu at (159.2, 88.2)
- added R3: prog, Resistor_THT:R_Axial_DIN0207_L6.3mm_D2.5mm_P10.16mm_Horizontal, B.Cu at (136.2, 115.5)
- added R4: 10k, Resistor_THT:R_Axial_DIN0207_L6.3mm_D2.5mm_P10.16mm_Horizontal, F.Cu at (113.9, 96.2)
- added R5: 470R, Resistor_THT:R_Axial_DIN0207_L6.3mm_D2.5mm_P10.16mm_Horizontal, B.Cu at (139.6, 105.4)
- added R6: 220R, Resistor_THT:R_Axial_DIN0207_L6.3mm_D2.5mm_P10.16mm_Horizontal, B.Cu at (150.4, 75.0)
- added R7: 10k, Resistor_THT:R_Axial_DIN0207_L6.3mm_D2.5mm_P10.16mm_Horizontal, B.Cu at (161.7, 105.0)
- added R8: 1k, Resistor_THT:R_Axial_DIN0207_L6.3mm_D2.5mm_P10.16mm_Horizontal, B.Cu at (157.4, 102.6)
- added SW1: EC11J12-15P30C-SW, BartLib_Encoder:EC11J12-15P30C-SW, F.Cu at (181.5, 107.2)
- added SW2: MFP 120, BartLib_Switch:MFP 120, F.Cu at (118.5, 101.2)
- added SW3: 6x6 13, Button_Switch_THT:SW_PUSH_6mm_H13mm, F.Cu at (113.5, 108.0)
- added U1: STM32G071KxT, Package_QFP:LQFP-32_7x7mm_P0.8mm, B.Cu at (141.5, 78.0)
- added U2: AF-02841BMR-B, BartLib_Display:LED 14.2mm, F.Cu at (162.5, 74.8)
- added U3: TC1185-3.3, Package_TO_SOT_SMD:SOT-23-5, B.Cu at (133.2, 89.1)
- added U4: MCP73831-2-OT, Package_TO_SOT_SMD:SOT-23-5, B.Cu at (114.7, 87.7)
- added Y1: 32k768, BartLib_Crystal:Crystal_D2.00mm_L6.00mm, F.Cu at (126.5, 89.7)
Routing:
- net +3V3: track 0.00 -> 142.6 mm, vias 0 -> 3
- net /MODE: track 0.00 -> 103.1 mm, vias 0 -> 2
- net Net-(R2-Pad1): track 0.00 -> 89.8 mm, vias 0 -> 8
- net Net-(R6-Pad1): track 0.00 -> 85.1 mm
- net /BUTTON2: track 0.00 -> 81.2 mm, vias 0 -> 6
- net /LED2: track 0.00 -> 72.8 mm, vias 0 -> 1
- net /ENC1: track 0.00 -> 67.3 mm, vias 0 -> 1
- net /ENC2: track 0.00 -> 58.9 mm, vias 0 -> 1
- net /LED1: track 0.00 -> 55.7 mm, vias 0 -> 1
- net Net-(D1-Pad1): track 0.00 -> 54.8 mm, vias 0 -> 1
- net /SYS_SWDIO: track 0.00 -> 54.8 mm, vias 0 -> 4
- net Net-(R3-Pad1): track 0.00 -> 54.7 mm, vias 0 -> 2
- net Net-(D3-Pad1): track 0.00 -> 53.0 mm
- net Net-(Q5-Pad2): track 0.00 -> 48.7 mm, vias 0 -> 2
- net /BUTTON1: track 0.00 -> 48.0 mm, vias 0 -> 1
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- added copper zone on B.Cu, net GND
- added copper zone on F.Cu, net GND
