File: doc/pcb/LEDthermowatch/LEDthermowatch.kicad_sch (KiCad schematic)
At the start: 63 parts, among them J1 Lipo

Commit message: drawn PCB
Parts:
- removed C?: 10u, symbol Device:C
- removed C?: 4u7, symbol Device:C
- removed H5: (no value), symbol Mechanical:MountingHole_Pad
- removed Q1, Q2, Q3, Q4: (no value), symbol Transistor_BJT:BC807
- removed Q6: (no value), symbol Device:Q_NMOS_GSD
- removed R12, R13, R15, R9: (no value), symbol Device:R
- added C3, C4: 10uF, Capacitor_THT:CP_Radial_D6.3mm_P2.50mm, symbol Device:C_Polarized
- added Q1, Q2, Q3, Q4: BC558, Package_TO_SOT_THT:TO-92, symbol Device:Q_PNP_CBE
- added Q5: 2N7000, Package_TO_SOT_THT:TO-92, symbol Device:Q_NMOS_SGD
- added R26, R27, R28, R29: 1k, Resistor_THT:R_Axial_DIN0207_L6.3mm_D2.5mm_P10.16mm_Horizontal, symbol Device:R
- C1, C2: renamed from C?; footprint (none) -> Capacitor_SMD:C_0805_2012Metric
- C15, C16, C17, C18, C19, C20, C6: value (none) -> 100n; footprint (none) -> Capacitor_SMD:C_0805_2012Metric
- C7: value (none) -> 1u; footprint (none) -> Capacitor_THT:CP_Radial_D6.3mm_P2.50mm
- C8, C9: value (none) -> 10p; footprint (none) -> Capacitor_SMD:C_0805_2012Metric
- D1: renamed from D?; footprint (none) -> LED_SMD:LED_0805_2012Metric
- D2: value (none) -> LED2; footprint (none) -> LED_SMD:LED_0805_2012Metric
- D3: value (none) -> LED1; footprint (none) -> LED_SMD:LED_0805_2012Metric
- H1, H2, H3, H4: value (none) -> MountingHole_Pad; footprint (none) -> BartLib_Pad:WirePad 4mm^2 Rect
- J1: value Lipo -> Lipo L503040; footprint (none) -> BartLib_Battery:CELLEVIA 30x40mm
- J2: value (none) -> SWD; footprint (none) -> Connector_PinHeader_2.54mm:PinHeader_1x05_P2.54mm_Vertical
- J3: renamed from J?; footprint (none) -> Connector_USB:USB_Micro-B_Molex_47346-0001
- R1, R4, R7: value (none) -> 10k; footprint (none) -> Resistor_THT:R_Axial_DIN0207_L6.3mm_D2.5mm_P10.16mm_Horizontal
- R10, R11: value (none) -> 220; footprint (none) -> Resistor_THT:R_Axial_DIN0207_L6.3mm_D2.5mm_P10.16mm_Horizontal
- R14, R2, R6: value (none) -> 220R; footprint (none) -> Resistor_THT:R_Axial_DIN0207_L6.3mm_D2.5mm_P10.16mm_Horizontal
- R16, R17, R8: value (none) -> 1k; footprint (none) -> Resistor_THT:R_Axial_DIN0207_L6.3mm_D2.5mm_P10.16mm_Horizontal
- R18, R19, R20, R21, R22, R23, R24, R25: value (none) -> 470R; footprint (none) -> Resistor_SMD:R_0805_2012Metric
- R3, R5: renamed from R?; footprint (none) -> Resistor_THT:R_Axial_DIN0207_L6.3mm_D2.5mm_P10.16mm_Horizontal
- SW1: value (none) -> EC11J12-15P30C-SW; footprint (none) -> BartLib_Encoder:EC11J12-15P30C-SW
- SW2: value (none) -> MFP 120; footprint (none) -> BartLib_Switch:MFP 120
- SW3: value (none) -> 6x6 13; footprint (none) -> Button_Switch_THT:SW_PUSH_6mm_H13mm
- U1: value (none) -> STM32G071KxT; footprint (none) -> Package_QFP:LQFP-32_7x7mm_P0.8mm
- U2: value (none) -> AF-02841BMR-B; footprint (none) -> BartLib_Display:LED 14.2mm
- Y1: value (none) -> 32k768; footprint (none) -> BartLib_Crystal:Crystal_D2.00mm_L6.00mm
- gave numbers to parts that had none: 2
Connections:
- net +3V3: now also C3.1, Q1.1 (C), Q2.1 (C), Q3.1 (C), Q4.1 (C)
- net +5V: now also C4.1
- net DISP_0: now also R26.1
- net DISP_1: now also R27.1
- net DISP_2: now also R28.1
- net DISP_3: now also R29.1
- net GND: now also C3.2, C4.2, Q5.1 (S)
- net at R8.2: now also Q5.2 (G)
- net at U2.12 (CC1): now also Q1.3 (E)
- net at U2.6 (CC4): now also Q4.3 (E)
- net at U2.8 (CC3): now also Q3.3 (E)
- net at U2.9 (CC2): now also Q2.3 (E)
- net at SW1.C: now also Q5.3 (D)
- new net: Q2.2 (B), R27.2
- new net: Q1.2 (B), R26.2
- new net: Q4.2 (B), R29.2
- new net: Q3.2 (B), R28.2
- no-connect marks 12 -> 11
Other:
- note removed: "CONRTOL BY MCU"
- note removed: "FORCE ACTIVE"
- moved on the sheet: H1, H2, H3, H4
